File: FidgetSpinner-PCB/FidgetSpinner.sch (KiCad schematic (older format))
At the start: 37 parts, among them J1 EdgeConnector, J2 GP2S27, SW1 SW_POWER, SW2 button, U1 STM32L010K8T6

Commit message: removed edge connector
Parts:
- removed J1: EdgeConnector, WYW_Package:Edge_2x05_2.54, symbol Connector_Generic:Conn_01x05
- added J1: DBG_CONN, Connector_PinHeader_2.54mm:PinHeader_1x06_P2.54mm_Horizontal, symbol Connector:Conn_01x06_Male
Connections:
- wire segments 124 -> 130
Changed lines of the file:
@@
 	1    0    0    -1
 $EndComp
-Text GLabel 7350 5550 0    50   BiDi ~ 0
+Text GLabel 7350 5650 0    50   BiDi ~ 0
 SWEN
-$Comp
-L Connector_Generic:Conn_01x05 J1
-U 1 1 6136C921
-P 7550 5350
-F 0 "J1" H 7630 5392 50  0000 L CNN
-F 1 "EdgeConnector" H 7630 5301 50  0000 L CNN
-F 2 "WYW_Package:Edge_2x05_2.54" H 7550 5350 50  0001 C CNN
-F 3 "~" H 7550 5350 50  0001 C CNN
-	1    7550 5350
-	1    0    0    -1
-$EndComp
 Text GLabel 4050 4750 2    50   BiDi ~ 0
 SWDIO
@@
 Wire Wire Line
 	7400 2100 7400 2250
+$Comp
+L Connector:Conn_01x06_Male J1
+U 1 1 61518390
+P 7700 5350
+F 0 "J1" H 7672 5324 50  0000 R CNN
+F 1 "DBG_CONN" H 7672 5233 50  0000 R CNN
+F 2 "Connector_PinHeader_2.54mm:PinHeader_1x06_P2.54mm_Horizontal" H 7700 5350 50  0001 C CNN
+F 3 "~" H 7700 5350 50  0001 C CNN
+	1    7700 5350
+	-1   0    0    -1
+$EndComp
+$Comp
+L power:VCC #PWR0111
+U 1 1 615233D8
+P 7350 5550
+F 0 "#PWR0111" H 7350 5400 50  0001 C CNN
+F 1 "VCC" V 7350 5750 50  0000 C CNN
+F 2 "" H 7350 5550 50  0001 C CNN
+F 3 "" H 7350 5550 50  0001 C CNN
+	1    7350 5550
+	0    -1   -1   0
+$EndComp
+Wire Wire Line
+	7350 5150 7500 5150
+Wire Wire Line
+	7350 5250 7500 5250
+Wire Wire Line
+	7350 5350 7500 5350
+Wire Wire Line
+	7350 5450 7500 5450
+Wire Wire Line
+	7350 5550 7500 5550
+Wire Wire Line
+	7350 5650 7500 5650
 $EndSCHEMATC

Commit message: bug fixes
Parts:
- removed J2: GP2S27, WYW_Package:4pin_5040, symbol Connector_Generic:Conn_02x02_Counter_Clockwise
- added R15: 2M, Resistor_SMD:R_0805_2012Metric_Pad1.20x1.40mm_HandSolder, symbol Device:R_Small
- added U2: GP2S60, WYW_Package:GP2S60_3217, symbol WYW_Library:GP2S60
- R10: value R_IR -> 33k
Connections:
- net GND: now also U2.2 (Rx-), U2.3 (Tx-)
- net VCC: now also R10.1, R15.2; no longer R10.2
- net ~INT_C: now also R15.1, U2.1 (Rx+)
- new net: R10.2, U2.4 (Tx+)
Other:
- note added: "Button"
- note removed: "Human Interface"
- moved on the sheet: C8, D10, D11, D12, D13, D14, D15, D16, D17, J1, R1, R10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

Commit message: backup
Parts:
- added R13, R14: ?M, Resistor_SMD:R_0805_2012Metric_Pad1.20x1.40mm_HandSolder, symbol Device:R_Small
- added U3: TS881, Package_TO_SOT_SMD:SOT-353_SC-70-5, symbol Amplifier_Operational:TS881xCx
- R15: value 2M -> ?M
Connections:
- net GND: now also R14.1, U3.2 (V-)
- net VCC: now also R13.1, U3.5 (V+)
- net ~INT_C renamed IR_OUT
- net IR_OUT: now also U3.3 (+); no longer U1.22 (PA12)
- new net: R13.2, R14.2, U3.4 (-)
- new net INT_C: U1.22 (PA12), U3.1
Other:
- moved on the sheet: C8, D10, D11, D12, D13, D14, D15, D16, D17, J1, R1, R2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
